Commit message: update robot_core.xacro

File: description/robot_core.xacro (robot description, xacro)
@@ -13,3 +13,19 @@
     <color rgba="0 0 0 1"/>
 </material>
+<link name="base_link">
+</link>
+<joint name="chassis_joint" type="fixed">
+    <parent link="base_link"/>
+    <child link="chassis"/>
+    <origin xyz="-0.1 0 0"/>
+</joint>
+<link name="chassis">
+    <visual>
+        <origin xyz="0.15 00.075" rpy="0 0 0"/>
+        <geometry>
+            <box size="0.3 0.3 0.15"/>
+        </geometry>
+        <material name="white"/>
+    </visual>
+</link>
 </robot>

Commit message: add wheels

File: description/robot_core.xacro (robot description, xacro)
@@ -15,4 +15,5 @@
 <link name="base_link">
 </link>
+<!-- CHASSIS-->
 <joint name="chassis_joint" type="fixed">
     <parent link="base_link"/>
@@ -22,5 +23,5 @@
 <link name="chassis">
     <visual>
-        <origin xyz="0.15 00.075" rpy="0 0 0"/>
+        <origin xyz="0.15 0 0.075" rpy="0 0 0"/>
         <geometry>
             <box size="0.3 0.3 0.15"/>
@@ -29,3 +30,33 @@
     </visual>
 </link>
+<!-- LEFT WHEEL-->
+<joint name="left_wheel_joint" type="continuous">
+    <parent link="base_link"/>
+    <child link="left_wheel"/>
+    <origin xyz="0 0.175 0" rpy="-${pi/2} 0 0"/>
+    <axis xyz="0 0 1"/>
+</joint>
+<link name="left_wheel">
+    <visual>
+        <geometry>
+            <cylinder length="0.04" radius="0.05" />
+        </geometry>
+        <material name="blue"/>
+    </visual>
+</link>
+<!-- RIGHT WHEEL-->
+<joint name="right_wheel_joint" type="continuous">
+    <parent link="base_link"/>
+    <child link="right_wheel"/>
+    <origin xyz="0 0.175 0" rpy="${pi/2} 0 0"/>
+    <axis xyz="0 0 -1"/>
+</joint>
+<link name="right_wheel">
+    <visual>
+        <geometry>
+            <cylinder length="0.04" radius="0.05" />
+        </geometry>
+        <material name="blue"/>
+    </visual>
+</link>
 </robot>

Commit message: fix typo wheel xacro

File: description/robot_core.xacro (robot description, xacro)
@@ -49,5 +49,5 @@
     <parent link="base_link"/>
     <child link="right_wheel"/>
-    <origin xyz="0 0.175 0" rpy="${pi/2} 0 0"/>
+    <origin xyz="0 -0.175 0" rpy="${pi/2} 0 0"/>
     <axis xyz="0 0 -1"/>
 </joint>
@@ -60,3 +60,17 @@
     </visual>
 </link>
+<!-- CASTER WHEEL -->
+<joint name="caster_wheel_joint" type="fixed">
+    <parent link="chassis"/>
+    <child link="caster_wheel"/>
+    <origin xyz="0.24 0 0" rpy="0 0 0"/>
+</joint>
+<link name="caster_wheel">
+    <visual>
+        <geometry>
+            <sphere radius="0.05" />
+        </geometry>
+        <material name="black"/>
+    </visual>
+</link>
 </robot>

Commit message: add xacro property

File: description/robot_core.xacro (robot description, xacro)
@@ -1,4 +1,5 @@
 <?xml version="1.0"?>
 <robot xmlns:xacro="https://www.ros.org/wiki/xacro">
+<!-- COLOR PARAMETERS-->
 <material name="white">
     <color rgba="1 1 1 1"/>
@@ -13,4 +14,19 @@
     <color rgba="0 0 0 1"/>
 </material>
+<!--PROPERTIES-->
+<xacro:property name="caster_wheel_radius" value="0.05"/>
+<xacro:property name="caster_wheel_origin_xyz" value="0.24 0 0"/>
+<xacro:property name="caster_wheel_origin_rpy" value="0 0 0"/>
+<xacro:property name="left_wheel_radius" value="0.05"/>
+<xacro:property name="left_wheel_length" value="0.05"/>
+<xacro:property name="left_wheel_origin_xyz" value="0 -0.175 0"/>
+<xacro:property name="left_wheel_origin_rpy" value="-${pi/2} 0 0"/>
+<xacro:property name="right_wheel_radius" value="0.05"/>
+<xacro:property name="right_wheel_length" value="0.05"/>
+<xacro:property name="right_wheel_origin_xyz" value="0 -0.175 0"/>
+<xacro:property name="right_wheel_origin_rpy" value="${pi/2} 0 0"/>
+<xacro:property name="chassis_origin_xyz" value="0.15 0 0.075"/>
+<xacro:property name="chassis_origin_rpy" value="0 0 0"/>
+<xacro:property name="chassis_joint_origin_xyz" value="-0.1 0 0"/>
 <link name="base_link">
 </link>
@@ -29,4 +45,10 @@
         <material name="white"/>
     </visual>
+    <collision>
+        <origin xyz="0.15 0 0.075" rpy="0 0 0"/>
+        <geometry>
+            <box size="0.3 0.3 0.15"/>
+        </geometry>
+    </collision>
 </link>
 <!-- LEFT WHEEL-->
@@ -44,4 +66,10 @@
         <material name="blue"/>
     </visual>
+    <collision>
+        <origin xyz="0 0.175 0" rpy="-${pi/2} 0 0"/>
+        <geometry>
+            <cylinder length="0.04" radius="0.05" />
+        </geometry>
+    </collision>
 </link>
 <!-- RIGHT WHEEL-->
@@ -55,22 +83,35 @@
     <visual>
         <geometry>
-            <cylinder length="0.04" radius="0.05" />
+            <cylinder length="${right_wheel_length}" radius="${right_wheel_radius}" />
         </geometry>
         <material name="blue"/>
     </visual>
+    <collision>
+        <origin xyz="${right_wheel_origin_xyz}" rpy="${right_wheel_origin_rpy}"/>
+        <geometry>
+            <cylinder length="${right_wheel_length}" radius="${right_wheel_radius}" />
+        </geometry>
+    </collision>
 </link>
 <!-- CASTER WHEEL -->
+<xacro:property name="caster_wheel_radius" value="0.05"/>
 <joint name="caster_wheel_joint" type="fixed">
     <parent link="chassis"/>
     <child link="caster_wheel"/>
-    <origin xyz="0.24 0 0" rpy="0 0 0"/>
+    <origin xyz="${caster_wheel_origin_xyz}" rpy="${caster_wheel_origin_rpy}"/>
 </joint>
 <link name="caster_wheel">
     <visual>
         <geometry>
-            <sphere radius="0.05" />
+            <sphere radius="${caster_wheel_radius}"/>
         </geometry>
         <material name="black"/>
     </visual>
+    <collision>
+        <origin xyz="${caster_wheel_origin_xyz}" rpy="${caster_wheel_origin_rpy}"/>
+        <geometry>
+            <sphere radius="0.05"/>
+        </geometry>
+    </collision>
 </link>
 </robot>

Commit message: update xacro file

File: description/robot_core.xacro (robot description, xacro)
@@ -20,5 +20,5 @@
 <xacro:property name="left_wheel_radius" value="0.05"/>
 <xacro:property name="left_wheel_length" value="0.05"/>
-<xacro:property name="left_wheel_origin_xyz" value="0 -0.175 0"/>
+<xacro:property name="left_wheel_origin_xyz" value="0 0.175 0"/>
 <xacro:property name="left_wheel_origin_rpy" value="-${pi/2} 0 0"/>
 <xacro:property name="right_wheel_radius" value="0.05"/>
@@ -29,4 +29,5 @@
 <xacro:property name="chassis_origin_rpy" value="0 0 0"/>
 <xacro:property name="chassis_joint_origin_xyz" value="-0.1 0 0"/>
+<xacro:property name="chassis_dimensions" value="0.3 0.3 0.15"/>
 <link name="base_link">
 </link>
@@ -35,5 +36,5 @@
     <parent link="base_link"/>
     <child link="chassis"/>
-    <origin xyz="-0.1 0 0"/>
+    <origin xyz="${chassis_joint_origin_xyz}"/>
 </joint>
 <link name="chassis">
@@ -41,12 +42,12 @@
         <origin xyz="0.15 0 0.075" rpy="0 0 0"/>
         <geometry>
-            <box size="0.3 0.3 0.15"/>
+            <box size="${chassis_dimensions}"/>
         </geometry>
-        <material name="white"/>
+        <material name="orange"/>
     </visual>
     <collision>
-        <origin xyz="0.15 0 0.075" rpy="0 0 0"/>
+        <origin xyz="${chassis_origin_xyz}" rpy="${chassis_origin_rpy}"/>
         <geometry>
-            <box size="0.3 0.3 0.15"/>
+            <box size="${chassis_dimensions}"/>
         </geometry>
     </collision>
@@ -56,5 +57,5 @@
     <parent link="base_link"/>
     <child link="left_wheel"/>
-    <origin xyz="0 0.175 0" rpy="-${pi/2} 0 0"/>
+    <origin xyz="${left_wheel_origin_xyz}" rpy="${left_wheel_origin_rpy}"/>
     <axis xyz="0 0 1"/>
 </joint>
@@ -62,12 +63,12 @@
     <visual>
         <geometry>
-            <cylinder length="0.04" radius="0.05" />
+            <cylinder length="${left_wheel_length}" radius="${left_wheel_radius}" />
         </geometry>
         <material name="blue"/>
     </visual>
     <collision>
-        <origin xyz="0 0.175 0" rpy="-${pi/2} 0 0"/>
+        <origin xyz="${left_wheel_origin_xyz}" rpy="${left_wheel_origin_rpy}"/>
         <geometry>
-            <cylinder length="0.04" radius="0.05" />
+            <cylinder length="${left_wheel_length}" radius="${left_wheel_radius}" />
         </geometry>
     </collision>
@@ -77,5 +78,5 @@
     <parent link="base_link"/>
     <child link="right_wheel"/>
-    <origin xyz="0 -0.175 0" rpy="${pi/2} 0 0"/>
+    <origin xyz="${right_wheel_origin_xyz}" rpy="${right_wheel_origin_rpy}"/>
     <axis xyz="0 0 -1"/>
 </joint>

Commit message: add inertial xacro

File: description/robot_core.xacro (robot description, xacro)
@@ -1,4 +1,5 @@
 <?xml version="1.0"?>
 <robot xmlns:xacro="https://www.ros.org/wiki/xacro">
+<xacro:include filename="inertial_macros.xacro"/>
 <!-- COLOR PARAMETERS-->
 <material name="white">
@@ -52,4 +53,7 @@
         </geometry>
     </collision>
+    <xacro:inertial_box mass="0.5" x="0.3" y="0.3" z="0.15">
+        <origin xyz="${chassis_origin_xyz}" rpy="${chassis_origin_rpy}"/>
+    </xacro:inertial_box>
 </link>
 <!-- LEFT WHEEL-->
@@ -68,9 +72,11 @@
     </visual>
     <collision>
-        <origin xyz="${left_wheel_origin_xyz}" rpy="${left_wheel_origin_rpy}"/>
         <geometry>
             <cylinder length="${left_wheel_length}" radius="${left_wheel_radius}" />
         </geometry>
     </collision>
+    <xacro:inertial_cylinder mass="0.1" length="0.05" radius="0.05">
+        <origin xyz="0 0 0" rpy="0 0 0"/>
+    </xacro:inertial_cylinder>
 </link>
 <!-- RIGHT WHEEL-->
@@ -89,9 +95,11 @@
     </visual>
     <collision>
-        <origin xyz="${right_wheel_origin_xyz}" rpy="${right_wheel_origin_rpy}"/>
         <geometry>
             <cylinder length="${right_wheel_length}" radius="${right_wheel_radius}" />
         </geometry>
     </collision>
+    <xacro:inertial_cylinder mass="0.1" length="0.05" radius="0.05">
+        <origin xyz="0 0 0" rpy="0 0 0"/>
+    </xacro:inertial_cylinder>
 </link>
 <!-- CASTER WHEEL -->
@@ -110,9 +118,11 @@
     </visual>
     <collision>
-        <origin xyz="${caster_wheel_origin_xyz}" rpy="${caster_wheel_origin_rpy}"/>
         <geometry>
             <sphere radius="0.05"/>
         </geometry>
     </collision>
+    <xacro:inertial_sphere mass="0.1" radius="0.05">
+        <origin xyz="0 0 0" rpy="0 0 0"/>
+    </xacro:inertial_sphere>
 </link>
 </robot>

Commit message: add gazebo ref material

File: description/robot_core.xacro (robot description, xacro)
@@ -57,4 +57,7 @@
     </xacro:inertial_box>
 </link>
+<gazebo reference="chassis">
+    <material>Gazebo/Orange</material>
+</gazebo>
 <!-- LEFT WHEEL-->
 <joint name="left_wheel_joint" type="continuous">
@@ -80,4 +83,7 @@
     </xacro:inertial_cylinder>
 </link>
+<gazebo reference="left_wheel">
+    <material>Gazebo/Blue</material>
+</gazebo>
 <!-- RIGHT WHEEL-->
 <joint name="right_wheel_joint" type="continuous">
@@ -103,4 +109,7 @@
     </xacro:inertial_cylinder>
 </link>
+<gazebo reference="right_wheel">
+    <material>Gazebo/Blue</material>
+</gazebo>
 <!-- CASTER WHEEL -->
 <xacro:property name="caster_wheel_radius" value="0.05"/>
@@ -126,3 +135,6 @@
     </xacro:inertial_sphere>
 </link>
+<gazebo reference="caster_wheel">
+    <material>Gazebo/Black</material>
+</gazebo>
 </robot>
